File: kicad/kassutronics-vco-3340.kicad_pcb (KiCad board)
At the start: 2 copper layers, 39.3 x 106.5 mm, 78 parts, among them J1 JACK_2P, J12 JACK_2P, J2 JACK_2P, J3 JACK_2P, J4 JACK_2P, J5 JACK_2P, J6 JACK_2P, J7 JACK_2P, J8 JACK_2P, J9 PWR, Q1 MMBFJ201, U1 TL074, U2 AS3340, U3 79L05, U4 LP2950

Commit message: pre-cleaned v0.1
Parts:
- added J13: Top Left(C), Connector_PinHeader_2.54mm:PinHeader_1x03_P2.54mm_Vertical, B.Cu at (2.42, 14.2)
- added J14: Top Left(M), Connector_PinHeader_2.54mm:PinHeader_1x03_P2.54mm_Vertical, F.Cu at (42.4, 14.2)
- added J15: Top Right(C), Connector_PinHeader_2.54mm:PinHeader_1x04_P2.54mm_Vertical, B.Cu at (37.5, 17.8)
- added J16: Top Right (M), Connector_PinHeader_2.54mm:PinHeader_1x04_P2.54mm_Vertical, F.Cu at (77.5, 17.8)
- added J17: Bottom Left(C), Connector_PinHeader_2.54mm:PinHeader_1x03_P2.54mm_Vertical, B.Cu at (2.16, 36.1)
- added J18: Bottom Left(M), Connector_PinHeader_2.54mm:PinHeader_1x03_P2.54mm_Vertical, F.Cu at (42.2, 36.1)
- added J19: Bottom Right(C), Connector_PinHeader_2.54mm:PinHeader_1x03_P2.54mm_Vertical, B.Cu at (37.5, 51.3)
- added J20: Bottom Right(M), Connector_PinHeader_2.54mm:PinHeader_1x03_P2.54mm_Vertical, F.Cu at (77.5, 51.3)
- C1: footprint Capacitor_THT:C_Disc_D5.0mm_W2.5mm_P2.50mm -> Capacitor_THT:C_Rect_L4.6mm_W2.0mm_P2.50mm_MKS02_FKP02
- C10, C13: footprint Capacitor_SMD:CP_Elec_6.3x5.4_Nichicon -> Capacitor_THT:CP_Radial_D5.0mm_P2.00mm
- C11, C2, C3, C4, C5, C6, C8: footprint Capacitor_THT:C_Rect_L4.6mm_W2.0mm_P2.50mm_MKS02_FKP02 -> Capacitor_THT:C_Rect_L4.6mm_W3.0mm_P2.50mm_MKS02_FKP02
- J9: footprint Connector_PinHeader_1.00mm:PinHeader_2x05_P1.00mm_Vertical -> SamacSys_Parts:SHDR10W50P254_2X5_2020X850X920P
- RV1, RV2, RV6, RV7: footprint Potentiometer_THT:Potentiometer_Bourns_3296X_Horizontal -> Potentiometer_THT:Potentiometer_Bourns_3296W_Vertical
- U1: footprint Package_DIP:DIP-14_W10.16mm_LongPads -> Package_DIP:DIP-14_W7.62mm_LongPads
- moved R6 162.3 mm to (56.4, 74.4)
- moved R14 159.5 mm to (23.3, 50.4)
- moved R19 151.8 mm to (10.9, 60.7)
- moved U3 149.4 mm to (56.7, 14.5), turned to 90 degrees
- moved C2 147.8 mm to (52.1, 11.7), turned to -90 degrees
- moved R35 147.7 mm to (53.0, 38.6), turned to 180 degrees
- moved R39 141.8 mm to (15.5, 32.8)
- moved C14 141.4 mm to (66.6, 53.3)
- moved R9 140.5 mm to (44.6, 74.4)
- moved R27 138.4 mm to (45.4, 53.8)
- moved R23 137.2 mm to (10.9, 63.7)
- moved D1 135.6 mm to (76.2, 74.9), turned to 180 degrees
- moved R31 134.3 mm to (45.4, 41.6)
- moved R18 132.5 mm to (76.2, 66.0), turned to 180 degrees
- moved R3 131.6 mm to (23.2, 40.3)
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Connections:
- C14 pad 2: /SAW_RAW -> /BR2M
- C15 pad 2: /PULSE_RAW -> /BL3M
- C8 pad 2: Net-(C8-Pad2) -> /TR3C
- J8 pad TN: +5VA -> /TR2C
- R11 pad 2: /CV_NODE -> /TL3C
- R14 pad 2: /SAW_RAW -> /BR2C
- R19 pad 2: /CV_NODE -> /TL3C
- R22 pad 1: /SAW_RAW -> /BR2M
- R23 pad 2: /CV_NODE -> /TL3C
- R24 pad 1: Net-(C8-Pad2) -> /TR3M
- R26 pad 2: /PULSE_RAW -> /BL3C
- R3 pad 2: /TRI_RAW -> /BR3C
- R30 pad 1: /PULSE_RAW -> /BL3M
- R31 pad 1: +5VA -> /TR2M
- R31 pad 2: /PWM_IN -> /BL1M
- R33 pad 2: /PWM_IN -> /BL1C
- R35 pad 1: /PWM_IN -> /BL1M
- R36 pad 2: /PWM_IN -> /BL1M
- R38 pad 2: /SIN_RAW -> /TL2C
- R39 pad 2: /CV_NODE -> /TL3C
- R9 pad 1: /TRI_RAW -> /BR3M
- RV3 pad 1: +5VA -> /TR2C_5V
- RV4 pad 1: +5VA -> /TR2C
- RV6 pad 1: /TRI_RAW -> /BR3M
- S1 pad 1: /SOFT_SYNC -> /BR1C
- S1 pad 3: /HARD_SYNC -> /BL2C
- U1 pad 14: /PULSE_RAW -> /BL3M
- U1 pad 7: /TRI_RAW -> /BR3M
- U1 pad 8: /SAW_RAW -> /BR2M
- U2 pad 5: /PWM_IN -> /BL1M
- U2 pad 6: /HARD_SYNC -> /BL2M
- U2 pad 9: /SOFT_SYNC -> /BR1M
Routing:
- net +12VA: track 0.00 -> 150.1 mm
- net /TR2C_5V: track 0.00 -> 122.5 mm
- net -12VA: track 0.00 -> 106.3 mm
- net +5VA: track 0.00 -> 86.6 mm
- net /SIN: track 0.00 -> 78.2 mm
- net /BL3C: track 0.00 -> 74.5 mm
- net /TRI: track 0.00 -> 71.0 mm
- net /TL3C: track 0.00 -> 68.4 mm
- net /SIN_RAW: track 0.00 -> 65.0 mm
- net -5VA: track 0.00 -> 61.6 mm
- net /SAW: track 0.00 -> 58.6 mm
- net Net-(D3-Pad1): track 0.00 -> 56.8 mm
- net /PULSE: track 0.00 -> 56.2 mm
- net /TR3C: track 0.00 -> 55.1 mm
- net /TL2C: track 0.00 -> 47.6 mm
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- added copper zone on B.Cu, net GND
- added copper zone on F.Cu, net GND
Other:
- board size 39.3 x 106.5 mm -> 79.5 x 106.5 mm
