File: kicad/kassutronics-vco-3340.kicad_sch (KiCad schematic)
At the start: 78 parts

Commit message: pre-cleaned v0.1
Parts:
- added J13, J17, J19: (no value), symbol Connector:Conn_01x03_Female
- added J14, J18, J20: (no value), symbol Connector:Conn_01x03_Male
- added J15: (no value), symbol Connector:Conn_01x04_Female
- added J16: (no value), symbol Connector:Conn_01x04_Male
Connections:
- net +5VA: now also J16.2 (Pin_2); no longer J8.TN, R31.1, RV3.1, RV4.1
- net CV_NODE: now also J14.3 (Pin_3); no longer R11.2, R19.2, R23.2, R39.2
- net GND: now also J15.4 (Pin_4), J16.4 (Pin_4)
- net SIN_RAW: now also J14.2 (Pin_2); no longer R38.2
- net TR3C: now reaches C8.2
- net TR3C: now also J15.3 (Pin_3); no longer R24.1
- net HARD_SYNC renamed BL2C
- net BL2C: now also J17.2 (Pin_2); no longer U2.6 (VHSI)
- net PULSE_RAW renamed BL3M
- net BL3M: now also J18.3 (Pin_3); no longer R26.2
- net PWM_IN renamed BL1M
- net BL1M: now also J18.1 (Pin_1); no longer R33.2
- net SAW_RAW renamed BR2M
- net BR2M: now also J20.2 (Pin_2); no longer R14.2
- net SOFT_SYNC renamed BR1C
- net BR1C: now also J19.1 (Pin_1); no longer U2.9 (VSSI)
- net TRI_RAW renamed BR3M
- net BR3M: now also J20.3 (Pin_3); no longer R3.2
- new net BL1C: J17.1 (Pin_1), R33.2
- new net BL2M: J18.2 (Pin_2), U2.6 (VHSI)
- new net BL3C: J17.3 (Pin_3), R26.2
- new net BR1M: J20.1 (Pin_1), U2.9 (VSSI)
- new net BR2C: J19.2 (Pin_2), R14.2
- new net BR3C: J19.3 (Pin_3), R3.2
- new net TL1C: J13.1 (Pin_1)
- new net TL1M: J14.1 (Pin_1)
- new net TL2C: J13.2 (Pin_2), R38.2
- new net TL3C: J13.3 (Pin_3), R11.2, R19.2, R23.2, R39.2
- new net TR1C: J15.1 (Pin_1)
- new net TR1M: J16.1 (Pin_1)
- new net TR2C: J8.TN, RV4.1
- new net TR2C_5V: J15.2 (Pin_2), RV3.1
- new net TR2M: R31.1
- new net TR3M: J16.3 (Pin_3), R24.1
Other:
- moved on the sheet: C4, C5, J3, J5, R11, R13, R15, R19, R23, R24, R35, R39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
