File: hardware/control-board/control-board.kicad_sch (KiCad schematic)
At the start: 28 parts

Commit message: Upgrade board files to KiCad 10 format
Ran kicad-cli sch upgrade and kicad-cli pcb upgrade across every board project.
Schematics move to 20260306, boards to 20260206, generator_version to 10.0.

The hardware/shared submodule pin moves to the matching eurorack-common-library
format upgrade — the two have to land together, since KiCad 9 cannot read either
side once migrated.

ERC reports 0 errors across all boards. Remaining warnings are lib_symbol_mismatch
against cached copies and pre-existing design warnings, neither introduced here.

Co-Authored-By: Claude Opus 5 (1M context) <noreply@anthropic.com>
Parts:
- J1, J12, J14, J16, J18, J2, J20, J3, J4, J5, J6, J7, J8: value ~ -> (none)
