File: hardware/main-board/main-board.kicad_sch (KiCad schematic)
At the start: 58 parts, among them Q1 MMBFJ201, U1 TL074, U2 AS3340, U3 79L05, U4 LP2950

Commit message: Upgrade board files to KiCad 10 format
Ran kicad-cli sch upgrade and kicad-cli pcb upgrade across every board project.
Schematics move to 20260306, boards to 20260206, generator_version to 10.0.

The hardware/shared submodule pin moves to the matching eurorack-common-library
format upgrade — the two have to land together, since KiCad 9 cannot read either
side once migrated.

ERC reports 0 errors across all boards. Remaining warnings are lib_symbol_mismatch
against cached copies and pre-existing design warnings, neither introduced here.

Co-Authored-By: Claude Opus 5 (1M context) <noreply@anthropic.com>
Parts:
- D1, D2, D3, J14, J16, J18, J20, J9: value ~ -> (none)
